File: Electron/V1/PCB/CurrentCost.sch (EAGLE design)
At the start: 17 parts, among them J1 RJ45, U2 ELECTRONDUALNAMED, U3 24LC512

Commit message: Improved measurements and added value for RJ45
Parts:
- J1: FARNELL (none) -> 1524544
Changed lines of the file:
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@@
 <part name="SUPPLY13" library="SparkFun-Aesthetics" deviceset="3.3V" device=""/>
 <part name="H3" library="holes" deviceset="MOUNT-HOLE" device="3.2" value="MOUNT-HOLE3.2"/>
-<part name="J1" library="SparkFun-Connectors" deviceset="RJ45-8" device="PTH" value="RJ45"/>
+<part name="J1" library="SparkFun-Connectors" deviceset="RJ45-8" device="PTH" value="RJ45">
+<attribute name="FARNELL" value="1524544"/>
+</part>
 <part name="SUPPLY3" library="SparkFun-Aesthetics" deviceset="3.3V" device=""/>
 <part name="GND6" library="SparkFun-Aesthetics" deviceset="DGND" device=""/>
@@
 <instance part="SUPPLY13" gate="G$1" x="10.16" y="35.56"/>
 <instance part="H3" gate="G$1" x="256.54" y="165.1"/>
-<instance part="J1" gate="JP1" x="144.78" y="50.8"/>
+<instance part="J1" gate="JP1" x="144.78" y="50.8">
+<attribute name="FARNELL" x="144.78" y="50.8" size="1.778" layer="96" display="off"/>
+</instance>
 <instance part="SUPPLY3" gate="G$1" x="129.54" y="60.96"/>
 <instance part="GND6" gate="G$1" x="124.46" y="50.8" rot="R270"/>
